File: balancer-board/IsolatedCharger.sch (KiCad schematic (older format))
At the start: 7 parts, among them Q8 AO3400, U2 HJT622, U3 TP4056

Commit message: multiple changes
Parts:
- Q8: value AO3400 -> BSS123
Changed lines of the file:
@@
 $Descr A4 11693 8268
 encoding utf-8
-Sheet 6 9
+Sheet 2 9
 Title ""
 Date ""
@@
 AR Path="/5D97C89E/5D8FDF4A" Ref="U?"  Part="1"
 AR Path="/5D97C8A5/5D8FDF4A" Ref="U?"  Part="1"
-F 0 "U11" H 6500 3237 60  0000 C CNN
+F 0 "U3" H 6500 3237 60  0000 C CNN
 F 1 "TP4056" H 6500 3131 60  0000 C CNN
 F 2 "Package_SO:SOP-8_3.76x4.96mm_P1.27mm" H 6500 2700 60  0001 C CNN
@@
 AR Path="/5D97C89E/5D8FDF57" Ref="D?"  Part="1"
 AR Path="/5D97C8A5/5D8FDF57" Ref="D?"  Part="1"
-F 0 "D5" V 5246 2532 50  0000 R CNN
+F 0 "D1" V 5246 2532 50  0000 R CNN
 F 1 "Yellow" V 5155 2532 50  0000 R CNN
 F 2 "LED_THT:LED_D5.0mm_Horizontal_O1.27mm_Z15.0mm" V 5200 2600 50  0001 C CNN
@@
 AR Path="/5D97C89E/5D8FDF5D" Ref="R?"  Part="1"
 AR Path="/5D97C8A5/5D8FDF5D" Ref="R?"  Part="1"
-F 0 "R9" V 5846 2750 50  0000 C CNN
+F 0 "R1" V 5846 2750 50  0000 C CNN
 F 1 "330" V 5755 2750 50  0000 C CNN
 F 2 "Resistor_SMD:R_0805_2012Metric" H 5650 2750 50  0001 C CNN
@@
 AR Path="/5D97C89E/5D8FDF6A" Ref="R?"  Part="1"
 AR Path="/5D97C8A5/5D8FDF6A" Ref="R?"  Part="1"
-F 0 "R10" H 7159 3046 50  0000 L CNN
+F 0 "R2" H 7159 3046 50  0000 L CNN
 F 1 "1k5" H 7159 2955 50  0000 L CNN
 F 2 "Resistor_SMD:R_0805_2012Metric" H 7100 3000 50  0001 C CNN
@@
 AR Path="/5D97C89E/5D8FDF51" Ref="U?"  Part="1"
 AR Path="/5D97C8A5/5D8FDF51" Ref="U?"  Part="1"
-F 0 "U10" H 3850 3265 50  0000 C CNN
+F 0 "U2" H 3850 3265 50  0000 C CNN
 F 1 "HJT622" H 3850 3174 50  0000 C CNN
 F 2 "footprints:HJT622" H 3500 2900 50  0001 C CNN
@@
 AR Path="/5D921BF3/5D91335F" Ref="Q6"  Part="1"
 AR Path="/5D921BFA/5D91335F" Ref="Q7"  Part="1"
-F 0 "Q5" H 2806 2696 50  0000 L CNN
-F 1 "AO3400" H 2806 2605 50  0000 L CNN
+F 0 "Q1" H 2806 2696 50  0000 L CNN
+F 1 "BSS123" H 2806 2605 50  0000 L CNN
 F 2 "Package_TO_SOT_SMD:SOT-23" H 2800 2750 50  0001 C CNN
 F 3 "~" H 2600 2650 50  0001 C CNN
@@
 AR Path="/5D921BFA/5D919D60" Ref="C7"  Part="1"
 AR Path="/5D921C01/5D919D60" Ref="C8"  Part="1"
-F 0 "C5" H 7665 2846 50  0000 L CNN
+F 0 "C1" H 7665 2846 50  0000 L CNN
 F 1 "10uF" H 7665 2755 50  0000 L CNN
 F 2 "Capacitor_SMD:C_0805_2012Metric" H 7588 2650 50  0001 C CNN

Commit message: v0.1
Parts:
- Q8: symbol Device:Q_NMOS_GSD -> Transistor_FET:BSS123
Changed lines of the file:
@@
 	2700 2450 3200 2450
 $Comp
-L Device:Q_NMOS_GSD Q8
+L Transistor_FET:BSS123 Q8
 U 1 1 5D91335F
 P 2600 2650
