File: balancer-board/balancer.kicad_pcb (KiCad board)
At the start: 2 copper layers, 100 x 83 mm, 86 parts, among them J1 Conn_01x08_Male, J2 Conn_01x17_Male, Q1 AO3400, Q2 AO3400, Q3 AO3400, Q4 AO3400, Q5 AO3400, Q6 AO3400, Q7 AO3400, Q8 AO3400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

Commit message: multiple changes
Other:
- board text added: "Balancer Module | Version 0.1"
- board text removed: "Version 1.0"
Changed lines of the file:
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@@
     )
   )
-  (gr_text "Version 1.0" (at 112.014 126.746) (layer F.SilkS)
-    (effects (font (size 1 1) (thickness 0.15)))
+  (gr_text "Balancer Module | Version 0.1" (at 107.3658 126.5682) (layer F.SilkS)
+    (effects (font (size 1 1) (thickness 0.15)) (justify left))
   )
   (gr_text B (at 167.894 46.99 270) (layer B.SilkS)

Commit message: multiple changes
Parts:
- added C9: 10nF, Capacitor_SMD:C_0805_2012Metric_Pad1.15x1.40mm_HandSolder, F.Cu at (148.5, 57.4)
- added R17: 1M, Resistor_SMD:R_0805_2012Metric_Pad1.15x1.40mm_HandSolder, F.Cu at (147.5, 60.2)
- D1, D2, D3, D4, D5, D6, D7, D8: footprint LED_THT:LED_D3.0mm -> LED_THT:LED_D5.0mm_Horizontal_O1.27mm_Z15.0mm
- REF**: moved to B.Cu
- U1: footprint footprints:SOP-14 -> footprints:SO-14
- moved D1 0.88 mm to (187.5, 125.3)
- moved D2 0.88 mm to (182.5, 125.3)
- moved D3 0.88 mm to (177.5, 125.3)
- moved D4 0.88 mm to (172.5, 125.3)
- moved D5 0.88 mm to (167.5, 125.3)
- moved D6 0.88 mm to (162.5, 125.3)
- moved D7 0.88 mm to (157.5, 125.3)
- moved D8 0.88 mm to (152.5, 125.3)
- moved U1 0.74 mm to (153.2, 63.6), turned to 90 degrees
- moved U10 0.45 mm to (114.6, 119.6)
- moved U12 0.45 mm to (114.6, 85.3)
- moved U14 0.45 mm to (87.9, 119.6)
- moved U16 0.45 mm to (87.9, 85.3)
- moved U2 0.45 mm to (168.0, 119.6)
- moved U4 0.45 mm to (168.0, 85.3)
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Routing:
- net Net-(D8-Pad2): track 10.9 -> 105.2 mm, vias 0 -> 1
- net Net-(D8-Pad1): track 1.86 -> 94.1 mm, vias 1 -> 2
- net Net-(D6-Pad2): track 11.0 -> 90.9 mm
- net Net-(D6-Pad1): track 1.84 -> 77.4 mm
- net Net-(D7-Pad2): track 11.6 -> 77.6 mm, vias 0 -> 1
- net Net-(D7-Pad1): track 1.71 -> 63.6 mm, vias 1 -> 2
- net Net-(D2-Pad1): track 1.69 -> 62.0 mm
- net Net-(D4-Pad1): track 1.92 -> 60.7 mm
- net Net-(D4-Pad2): track 10.8 -> 67.6 mm
- net Net-(D2-Pad2): track 10.2 -> 61.5 mm
- net Net-(D5-Pad2): track 11.8 -> 62.7 mm, vias 0 -> 1
- net Net-(D5-Pad1): track 1.97 -> 43.0 mm, vias 1 -> 2
- net Net-(D3-Pad2): track 10.4 -> 41.6 mm, vias 0 -> 1
- net Vin: track 260.6 -> 289.7 mm
- net Net-(D3-Pad1): track 1.92 -> 27.9 mm, vias 1 -> 2
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Other:
- board text added: "A1"
- board text added: "A2"
- board text added: "A3"
- board text added: "A4"
- board text added: "A5"
- board text added: "A6"
- board text added: "A7"
- board text added: "A8"
- board text added: "B10"
- board text added: "B11"
- board text added: "B12"
- board text added: "B13"
- board text added: "B14"
- board text added: "B15"
- board text added: "B16"
- board text added: "B9"

Commit message: v0.1
Other:
- board text added: "Balancer Module | Version 0.1 | 2019-11-11"
- board text removed: "Balancer Module | Version 0.1"
Changed lines of the file:
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@@
       (layerselection 0x010fc_ffffffff)
       (usegerberextensions false)
-      (usegerberattributes false)
+      (usegerberattributes true)
       (usegerberadvancedattributes false)
       (creategerberjobfile false)
@@
       (plotinvisibletext false)
       (padsonsilk false)
-      (subtractmaskfromsilk false)
+      (subtractmaskfromsilk true)
       (outputformat 1)
       (mirror false)
-      (drillshape 1)
+      (drillshape 0)
       (scaleselection 1)
-      (outputdirectory ""))
+      (outputdirectory "output/v0.1/"))
   )
   (net 0 "")
@@
       (effects (font (size 1 1) (thickness 0.15)))
     )
-    (fp_text user DISABLE (at 22.86 -17.78) (layer F.SilkS)
+    (fp_text user DISABLE (at 22.0091 -17.7546) (layer F.SilkS)
       (effects (font (size 1 1) (thickness 0.15)))
     )
@@
       (effects (font (size 1 1) (thickness 0.15)))
     )
-    (fp_text user -Vin (at 24.028275 -29.567148) (layer F.SilkS)
+    (fp_text user -Vin (at 23.2283 -29.5656) (layer F.SilkS)
       (effects (font (size 1 1) (thickness 0.15)))
     )
@@
       (effects (font (size 1 1) (thickness 0.15)))
     )
-    (fp_text user DISABLE (at 22.86 -17.78) (layer F.SilkS)
+    (fp_text user DISABLE (at 22.1361 -17.8308) (layer F.SilkS)
       (effects (font (size 1 1) (thickness 0.15)))
     )
@@
       (effects (font (size 1 1) (thickness 0.15)))
     )
-    (fp_text user -Vin (at 24.028275 -29.567148) (layer F.SilkS)
+    (fp_text user -Vin (at 23.0251 -29.7942) (layer F.SilkS)
       (effects (font (size 1 1) (thickness 0.15)))
     )
@@
     (effects (font (size 0.5 0.5) (thickness 0.1)))
   )
-  (gr_text "Balancer Module | Version 0.1" (at 107.3658 126.5682) (layer F.SilkS)
-    (effects (font (size 1 1) (thickness 0.15)) (justify left))
+  (gr_text "Balancer Module | Version 0.1 | 2019-11-11" (at 107.3404 126.0856) (layer F.SilkS)
+    (effects (font (size 0.9 0.9) (thickness 0.15)) (justify left))
   )
   (gr_text B (at 167.894 46.99 270) (layer B.SilkS)
