File: main-board/measurement.sch (KiCad schematic (older format))
At the start: 48 parts, among them J9 Conn_01x03_Female, U3 ADS1115IDGS, U4 MAX14921ECS+T

Commit message: multiple changes
Parts:
- removed C26: 10nF, Capacitor_SMD:C_0805_2012Metric, symbol Device:C_Small
- removed J9: Conn_01x03_Female, symbol Connector:Conn_01x03_Female
- removed R24, R25: 1k, Resistor_SMD:R_0805_2012Metric, symbol Device:R_Small
- added C29, C30: 100nF, Capacitor_SMD:C_0805_2012Metric, symbol Device:C_Small
- added C32: 0u1, Capacitor_SMD:C_0805_2012Metric, symbol Device:C_Small
- added C37: ?, Capacitor_SMD:C_0805_2012Metric, symbol Device:C_Small
- added J9: Conn_01x02_Female, Connector_PinHeader_2.54mm:PinHeader_1x02_P2.54mm_Vertical, symbol Connector:Conn_01x02_Female
- added R1, R2: 1K, Capacitor_SMD:C_0805_2012Metric, symbol Device:R_Small
- added R30: 100k, Capacitor_SMD:C_0805_2012Metric, symbol Device:R_Small
- C10, C11, C12, C13, C14, C15, C16, C17, C18, C19, C20, C21, C22, C23, C24, C9: value 1u2 -> 2u2
- C25, C27: value 10nF -> 100nF
- R26: value 1k -> 220
- R27: value 10k -> 1K; footprint Resistor_SMD:R_0805_2012Metric -> Capacitor_SMD:C_0805_2012Metric
- R28, R29: value 10k -> 100k; footprint Resistor_SMD:R_0805_2012Metric -> Capacitor_SMD:C_0805_2012Metric
Connections:
- net +3V3: now also C32.2
- net +5V: now also R30.1; no longer R27.1
- net +5VA: now also U4.13 (LDOIN)
- net AOUT: now also R26.2; no longer U3.4 (AIN0)
- net GND: now also C29.2, C30.2, C32.1; no longer C15.1, C27.2, C8.2, U4.11 (AGND)
- net T1: now also R1.1, R30.2; no longer R27.2, U4.9 (T1)
- net T2: now also R29.2, C29.1, R2.1; no longer R28.2, U4.8 (T2)
- net T3: now also R27.1, R28.2, C30.1; no longer C27.1, R26.1, R26.2, R29.2, U4.7 (T3)
- net VC0: now also C15.1
- net GNDA: now reaches U3.5 (AIN1)
- net GNDA: now also C27.2, C8.2, U4.11 (AGND)
- net at U3.6 (AIN2): now also C37.1, J9.2 (Pin_2)
- net at U3.7 (AIN3): now also C37.2, J9.1 (Pin_1)
- net at C6.1, R7.1, U4.14 (VP): no longer U4.13 (LDOIN)
- new net: C27.1, R26.1, U3.4 (AIN0)
- new net T1f: R1.2, U4.9 (T1)
- new net T2f: R2.2, U4.8 (T2)
- new net T3f: R27.2, U4.7 (T3)

Commit message: multiple changes
Parts:
- C32, C6: value 0u1 -> 100nF
- C37: value ? -> reserved
- U3: footprint Package_SO:TSSOP-10_3x3mm_P0.5mm -> Package_SO:MSOP-10_3x3mm_P0.5mm
Changed lines of the file:
@@
 AR Path="/5DCC161B/5DCE2DF4" Ref="C6"  Part="1"
 F 0 "C6" H 2942 3146 50  0000 L CNN
-F 1 "0u1" H 2942 3055 50  0000 L CNN
+F 1 "100nF" H 2942 3055 50  0000 L CNN
 F 2 "Capacitor_SMD:C_0805_2012Metric" H 2850 3100 50  0001 C CNN
 F 3 "~" H 2850 3100 50  0001 C CNN
@@
 F 0 "U3" H 2050 2500 50  0000 C CNN
 F 1 "ADS1115IDGS" H 2000 2400 50  0000 C CNN
-F 2 "Package_SO:TSSOP-10_3x3mm_P0.5mm" H 2300 1400 50  0001 C CNN
+F 2 "Package_SO:MSOP-10_3x3mm_P0.5mm" H 2300 1400 50  0001 C CNN
 F 3 "http://www.ti.com/lit/ds/symlink/ads1113.pdf" H 2250 1000 50  0001 C CNN
 	1    2300 1900
@@
 P 4250 2300
 F 0 "C32" H 4158 2254 50  0000 R CNN
-F 1 "0u1" H 4158 2345 50  0000 R CNN
+F 1 "100nF" H 4158 2345 50  0000 R CNN
 F 2 "Capacitor_SMD:C_0805_2012Metric" H 4250 2300 50  0001 C CNN
 F 3 "~" H 4250 2300 50  0001 C CNN
@@
 P 1600 2250
 F 0 "C37" H 1692 2296 50  0000 L CNN
-F 1 "?" H 1692 2205 50  0000 L CNN
+F 1 "reserved" H 1692 2205 50  0000 L CNN
 F 2 "Capacitor_SMD:C_0805_2012Metric" H 1600 2250 50  0001 C CNN
 F 3 "~" H 1600 2250 50  0001 C CNN
