File: main-board/main-board.kicad_pcb (KiCad board)
At the start: 2 copper layers, 100 x 98 mm, 125 parts, among them J1 Conn_01x08_Male, J10 Raspberry_Pi_2_3, J11 T1, J12 T2, J13 T3, J2 USB_B, J3 Ext 5V, J4 Power Supply, J5 SWD, J6 Conn_01x17_Female, J7 9-16, J8 0-8, SW1 SW_DIP_x01, U1 L78L33_SOT89, U2 STM32F072CBTx, U3 ADS1115IDGS, U4 MAX14921ECS+T

Commit message: multiple changes
Parts:
- removed F18: 2A, Resistor_SMD:R_2512_6332Metric
- removed J4: Power Supply, TerminalBlock_RND:TerminalBlock_RND_205-00287_1x02_P5.08mm_Horizontal
- removed PS1: StepDownModule, footprints:LM2596HV_Module
- removed the REF** at (97.3, 122.2)
- removed the REF** at (190.0, 121.7)
- removed the REF** at (96.7, 49.2)
- removed the REF** at (188.5, 49.5)
- removed SW1: SW_DIP_x01, Button_Switch_THT:SW_Slide_1P2T_CK_OS102011MS2Q
- removed TP11: PB8, TestPoint:TestPoint_THTPad_2.5x2.5mm_Drill1.2mm
- removed TP12: PB9, TestPoint:TestPoint_THTPad_2.5x2.5mm_Drill1.2mm
- added C29: 100nF, Capacitor_SMD:C_0805_2012Metric, F.Cu at (101.9, 104.8)
- added C30: 100nF, Capacitor_SMD:C_0805_2012Metric, F.Cu at (102.0, 113.5)
- added C31: 22u, Capacitor_SMD:C_1206_3216Metric, F.Cu at (132.1, 67.7)
- added C32: 0u1, Capacitor_SMD:C_0805_2012Metric, F.Cu at (127.1, 103.7)
- added C33: 0u1, Capacitor_SMD:C_0805_2012Metric_Pad1.15x1.40mm_HandSolder, F.Cu at (165.7, 104.5)
- added C34: 0u1, Capacitor_SMD:C_0805_2012Metric_Pad1.15x1.40mm_HandSolder, F.Cu at (170.9, 101.3)
- added C35: 22u, Capacitor_SMD:C_1206_3216Metric, F.Cu at (170.2, 94.3)
- added C36: 22u, Capacitor_SMD:C_1206_3216Metric, F.Cu at (167.6, 94.3)
- added C37: ?, Capacitor_SMD:C_0805_2012Metric, F.Cu at (143.9, 113.4)
- added D5: SMAJ5.0A, Diode_SMD:D_SMA_Handsoldering, F.Cu at (163.2, 96.9)
- added J9: Conn_01x02_Female, Connector_PinHeader_2.54mm:PinHeader_1x02_P2.54mm_Vertical, F.Cu at (159.4, 109.5)
- added JP2: Bootloader, Jumper:SolderJumper-2_P1.3mm_Open_RoundedPad1.0x1.5mm, F.Cu at (104.9, 69.4)
- added L1: LQH3C 220u, Inductor_SMD:L_1210_3225Metric_Pad1.42x2.65mm_HandSolder, F.Cu at (153.4, 102.7)
- added L2: BLM21PG600SN1, Inductor_SMD:L_1210_3225Metric_Pad1.42x2.65mm_HandSolder, F.Cu at (127.7, 66.7)
- added L3: 100u, Inductor_SMD:L_Fastron_PISR_Handsoldering, F.Cu at (179.1, 90.4)
- added PB0: PB8, TestPoint:TestPoint_THTPad_2.0x2.0mm_Drill1.0mm, F.Cu at (117.4, 97.9)
- added PB1: PB9, TestPoint:TestPoint_THTPad_2.0x2.0mm_Drill1.0mm, F.Cu at (117.4, 92.9)
- added Q1: AO3400, Package_TO_SOT_SMD:SOT-23, F.Cu at (138.6, 66.7)
- added R30: 100k, Capacitor_SMD:C_0805_2012Metric, F.Cu at (101.8, 92.6)
- added R31: 100m, Resistor_SMD:R_0805_2012Metric, F.Cu at (168.8, 90.9)
- added REF**: OSHW-Logo2_7.3x6mm_SilkScreen, Symbol:OSHW-Logo2_7.3x6mm_SilkScreen, F.Cu at (189.4, 92.2)
- added U5: MAX5035BASA, Package_SO:SOIC-8_3.9x4.9mm_P1.27mm, F.Cu at (170.8, 105.1)
- C10, C11, C12, C13, C14, C15, C16, C17, C18, C19, C20, C21, C22, C23, C24, C9: value 1u2 -> 2u2
- C25, C27: value 10nF -> 100nF
- C26: value 10nF -> 68u 100V; footprint Capacitor_SMD:C_0805_2012Metric -> Capacitor_THT:CP_Radial_D12.5mm_P5.00mm
- C5: value 1u -> 22u; footprint Capacitor_SMD:C_0805_2012Metric -> Capacitor_SMD:C_1206_3216Metric
- D4: value 1N4733 -> SS210A; footprint Diode_THT:D_DO-41_SOD81_P7.62mm_Horizontal -> Diode_SMD:D_SMA_Handsoldering
- F19: value 2A -> 1A
- J1: value Conn_01x08_Male -> ModuleConnector
- J11, J12, J13: footprint TerminalBlock_MetzConnect:TerminalBlock_MetzConnect_Type059_RT06303HBWC_1x03_P3.50mm_Horizontal -> TerminalBlock_MetzConnect:TerminalBlock_MetzConnect_Type059_RT06302HBWC_1x02_P3.50mm_Horizontal
- J3: value Ext 5V -> ShuntBoard; footprint TerminalBlock_RND:TerminalBlock_RND_205-00288_1x03_P5.08mm_Horizontal -> TerminalBlock_4Ucon:TerminalBlock_4Ucon_1x06_P3.50mm_Horizontal
- J6: value Conn_01x17_Female -> Battery
- R1, R2: value 20R -> 1K; footprint Resistor_SMD:R_0805_2012Metric -> Capacitor_SMD:C_0805_2012Metric
- R24, R25: value 1k -> 10k
- R26: value 1k -> 220
- R27: value 10k -> 1K; footprint Resistor_SMD:R_0805_2012Metric -> Capacitor_SMD:C_0805_2012Metric
- R28, R29: value 10k -> 100k; footprint Resistor_SMD:R_0805_2012Metric -> Capacitor_SMD:C_0805_2012Metric
- R4: value 120R -> 62R
- TP10: value PB7 -> GND; footprint TestPoint:TestPoint_THTPad_2.5x2.5mm_Drill1.2mm -> TestPoint:TestPoint_THTPad_2.0x2.0mm_Drill1.0mm
- TP13, TP14, TP15, TP16, TP17, TP18, TP19, TP2, TP21, TP22, TP23, TP3, TP6: footprint TestPoint:TestPoint_THTPad_2.5x2.5mm_Drill1.2mm -> TestPoint:TestPoint_THTPad_2.0x2.0mm_Drill1.0mm
- TP20: value PA3 -> PA15; footprint TestPoint:TestPoint_THTPad_2.5x2.5mm_Drill1.2mm -> TestPoint:TestPoint_THTPad_2.0x2.0mm_Drill1.0mm
- TP4: value PC13 -> 5V; footprint TestPoint:TestPoint_THTPad_2.5x2.5mm_Drill1.2mm -> TestPoint:TestPoint_THTPad_2.0x2.0mm_Drill1.0mm
- TP5: value PC14 -> 3V3; footprint TestPoint:TestPoint_THTPad_2.5x2.5mm_Drill1.2mm -> TestPoint:TestPoint_THTPad_2.0x2.0mm_Drill1.0mm
- TP7: value PB4 -> GND; footprint TestPoint:TestPoint_THTPad_2.5x2.5mm_Drill1.2mm -> TestPoint:TestPoint_THTPad_2.0x2.0mm_Drill1.0mm
- TP8: value PB5 -> PB2; footprint TestPoint:TestPoint_THTPad_2.5x2.5mm_Drill1.2mm -> TestPoint:TestPoint_THTPad_2.0x2.0mm_Drill1.0mm
- TP9: value PB6 -> GND; footprint TestPoint:TestPoint_THTPad_2.5x2.5mm_Drill1.2mm -> TestPoint:TestPoint_THTPad_2.0x2.0mm_Drill1.0mm
- moved R5 168.0 mm to (120.3, 100.2), turned to 180 degrees
- moved C3 167.6 mm to (109.1, 85.1), turned to 90 degrees
- moved F19 164.3 mm to (166.6, 87.9), turned to 180 degrees
- moved C2 158.2 mm to (111.9, 78.4), turned to 90 degrees
- moved D2 150.7 mm to (189.2, 140.5)
- moved C26 148.4 mm to (181.1, 105.1), turned to 270 degrees
- moved R4 144.1 mm to (186.7, 135.4), turned to 270 degrees
- moved J3 137.4 mm to (97.0, 85.6)
- moved C28 125.1 mm to (150.9, 87.9)
- moved D3 124.1 mm to (191.5, 119.4), turned to 180 degrees
- moved R24 119.7 mm to (135.8, 66.7)
- moved C4 118.4 mm to (123.0, 80.5)
- moved D4 118.2 mm to (169.6, 98.8), turned to 180 degrees
- moved R6 117.3 mm to (120.3, 102.2), turned to 180 degrees
- moved R26 112.6 mm to (133.2, 108.3), turned to 90 degrees
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Connections:
- C26 pad 1: /measurement/T2 -> Vin
- C27 pad 1: /measurement/T3 -> Net-(C27-Pad1)
- D4 pad 1: +5V -> Net-(C34-Pad2)
- F1 pad 1: /measurement/VC16 -> Vin
- J10 pad 10: Net-(J10-Pad10) -> /UART_TX
- J10 pad 3: /PI_SDA -> Net-(J10-Pad3)
- J10 pad 5: /PI_SCL -> Net-(J10-Pad5)
- J10 pad 6: GND -> Net-(J10-Pad6)
- J10 pad 8: Net-(J10-Pad8) -> /UART_RX
- J2 pad 2: Net-(J2-Pad2) -> /USB_DM
- J2 pad 3: Net-(J2-Pad3) -> /USB_DP
- J3 pad 1: Vin -> GND
- J3 pad 2: GND -> /EN_OUT
- J3 pad 3: Net-(F19-Pad1) -> /EN_IN
- J6 pad 17: /measurement/VC16 -> Vin
- R1 pad 1: /USB_DP -> /measurement/T1
- R1 pad 2: Net-(J2-Pad3) -> /measurement/T1f
- R2 pad 1: /USB_DM -> /measurement/T2
- R2 pad 2: Net-(J2-Pad2) -> /measurement/T2f
- R24 pad 1: /measurement/T1 -> /PI_ON
- R24 pad 2: /measurement/T1 -> GND
- R25 pad 1: /measurement/T2 -> +3V3
- R25 pad 2: /measurement/T2 -> Net-(JP2-Pad2)
- R26 pad 1: /measurement/T3 -> Net-(C27-Pad1)
- R26 pad 2: /measurement/T3 -> /measurement/AOUT
- R27 pad 1: +5V -> /measurement/T3
- R27 pad 2: /measurement/T1 -> /measurement/T3f
- R28 pad 2: /measurement/T2 -> /measurement/T3
- R29 pad 2: /measurement/T3 -> /measurement/T2
- R4 pad 1: Net-(R4-Pad1) -> /LED
- R7 pad 2: /measurement/VC16 -> Vin
- R8 pad 2: /measurement/VC16 -> Vin
- TP1 pad 1: Net-(TP1-Pad1) -> Net-(JP2-Pad2)
- TP10 pad 1: Net-(TP10-Pad1) -> GND
- TP4 pad 1: Net-(TP4-Pad1) -> +5V
- TP5 pad 1: Net-(TP5-Pad1) -> +3V3
- TP7 pad 1: Net-(TP7-Pad1) -> GND
- TP9 pad 1: Net-(TP9-Pad1) -> GND
- U2 pad 13: Net-(TP20-Pad1) -> /LED
- U2 pad 18: /CS_A -> Net-(PB0-Pad1)
- U2 pad 19: /CS_B -> Net-(PB1-Pad1)
- U2 pad 2: Net-(TP4-Pad1) -> /EN_IN
- U2 pad 20: /DSB -> Net-(TP8-Pad1)
- U2 pad 3: Net-(TP5-Pad1) -> /EN_OUT
- U2 pad 38: Net-(R4-Pad1) -> Net-(TP20-Pad1)
- U2 pad 39: /DSA -> /PI_ON
- U2 pad 40: Net-(TP7-Pad1) -> /CS_B
- U2 pad 41: Net-(TP8-Pad1) -> /CS_A
- U2 pad 42: Net-(TP9-Pad1) -> /UART_TX
- U2 pad 43: Net-(TP10-Pad1) -> /UART_RX
- U2 pad 44: Net-(TP1-Pad1) -> Net-(JP2-Pad2)
- U2 pad 45: /PI_SCL -> /DSB
- U2 pad 46: /PI_SDA -> /DSA
- U3 pad 4: /measurement/AOUT -> Net-(C27-Pad1)
- U3 pad 5: Net-(J9-Pad3) -> GND
- U4 pad 13: Net-(C6-Pad1) -> +5VA
- U4 pad 7: /measurement/T3 -> /measurement/T3f
- U4 pad 8: /measurement/T2 -> /measurement/T2f
- U4 pad 9: /measurement/T1 -> /measurement/T1f
Routing:
- net GND: track 55.7 -> 360.1 mm, vias 0 -> 4
- net +5V: track 0.00 -> 252.5 mm, vias 0 -> 6
- net Vin: track 0.00 -> 243.4 mm
- net /LED: track 0.00 -> 179.6 mm, vias 0 -> 2
- net +3V3: track 22.9 -> 147.9 mm
- net /SDA: track 0.00 -> 94.7 mm, vias 0 -> 4
- net /SCL: track 0.00 -> 93.8 mm, vias 0 -> 4
- net /CS_B: track 0.00 -> 67.0 mm
- net /measurement/T1f: track 0.00 -> 64.5 mm, vias 0 -> 4
- net /CS_A: track 0.00 -> 64.4 mm
- net /DSB: track 0.00 -> 63.1 mm
- net /DSA: track 0.00 -> 61.8 mm
- net /measurement/T2f: track 0.00 -> 58.0 mm, vias 0 -> 2
- net /measurement/T3f: track 0.00 -> 49.3 mm, vias 0 -> 2
- net /PI_ON: track 0.00 -> 39.4 mm, vias 0 -> 2
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Other:
- board text added: "3V3"
- board text added: "5V"
- board text added: "5VA"
- board text added: "Controller Module | Version 0.1"
- board text added: "github.com/alangecker/yabalancer"
- board text removed: "Temperature"

Commit message: multiple changes
Parts:
- removed REF**: OSHW-Logo2_7.3x6mm_SilkScreen, Symbol:OSHW-Logo2_7.3x6mm_SilkScreen
- removed TP20: PA15, TestPoint:TestPoint_THTPad_2.0x2.0mm_Drill1.0mm
- removed TP23: PA10, TestPoint:TestPoint_THTPad_2.0x2.0mm_Drill1.0mm
- removed TP6: PC15, TestPoint:TestPoint_THTPad_2.0x2.0mm_Drill1.0mm
- added H1: MountingHole, MountingHole:MountingHole_3.2mm_M3_DIN965_Pad, F.Cu at (96.7, 49.2)
- added H2: MountingHole, MountingHole:MountingHole_3.2mm_M3_DIN965_Pad, F.Cu at (97.3, 122.2)
- added H3: MountingHole, MountingHole:MountingHole_3.2mm_M3_DIN965_Pad, F.Cu at (188.5, 49.5)
- added H4: MountingHole, MountingHole:MountingHole_3.2mm_M3_DIN965_Pad, F.Cu at (190.0, 121.7)
- added J4: ShuntBoard, Connector_JST:JST_XH_S6B-XH-A_1x06_P2.50mm_Horizontal, F.Cu at (97.9, 74.2)
- added R32: 2k2, Resistor_SMD:R_0805_2012Metric, F.Cu at (104.4, 79.5)
- added R33: 2k2, Resistor_SMD:R_0805_2012Metric, F.Cu at (109.9, 74.7)
- C32, C6: value 0u1 -> 100nF
- C33, C34: value 0u1 -> 100nF; footprint Capacitor_SMD:C_0805_2012Metric_Pad1.15x1.40mm_HandSolder -> Capacitor_SMD:C_0805_2012Metric
- C35, C36: footprint Capacitor_SMD:C_1206_3216Metric -> Capacitor_SMD:C_1210_3225Metric_Pad1.42x2.65mm_HandSolder
- C37: value ? -> reserved
- F1, F10, F11, F12, F13, F14, F15, F16, F19, F2, F3, F4, F5, F6, F7, F8, F9: footprint Resistor_SMD:R_2512_6332Metric -> Resistor_SMD:R_1812_4532Metric_Pad1.30x3.40mm_HandSolder
- F17: value 2A -> 1A; footprint Resistor_SMD:R_2512_6332Metric -> Resistor_SMD:R_1812_4532Metric_Pad1.30x3.40mm_HandSolder
- J11, J12, J13: footprint TerminalBlock_MetzConnect:TerminalBlock_MetzConnect_Type059_RT06302HBWC_1x02_P3.50mm_Horizontal -> Connector_JST:JST_XH_S2B-XH-A_1x02_P2.50mm_Horizontal
- J2: value USB_B -> USB
- J3: footprint TerminalBlock_4Ucon:TerminalBlock_4Ucon_1x06_P3.50mm_Horizontal -> Connector_JST:JST_XH_S6B-XH-A_1x06_P2.50mm_Horizontal
- JP2: value Bootloader -> Boot
- L2: footprint Inductor_SMD:L_1210_3225Metric_Pad1.42x2.65mm_HandSolder -> Inductor_SMD:L_0805_2012Metric_Pad1.15x1.40mm_HandSolder
- U3: footprint Package_SO:TSSOP-10_3x3mm_P0.5mm -> Package_SO:MSOP-10_3x3mm_P0.5mm
- U5: footprint Package_SO:SOIC-8_3.9x4.9mm_P1.27mm -> Package_SO:SOP-8_3.76x4.96mm_P1.27mm
- moved F17 86.7 mm to (183.6, 130.4)
- moved J3 29.9 mm to (97.9, 55.8), turned to 270 degrees
- moved C32 6.18 mm to (131.1, 108.4), turned to 90 degrees
- moved C34 5.97 mm to (165.0, 100.3)
- moved D3 5.21 mm to (191.5, 114.2)
- moved D1 5.21 mm to (191.5, 117.1)
- moved L2 3.83 mm to (130.8, 64.5)
- moved JP2 3.55 mm to (108.5, 69.6), turned to 90 degrees
- moved C7 3.40 mm to (137.5, 111.0)
- moved R25 3.04 mm to (110.8, 69.6)
- moved TP1 2.76 mm to (109.6, 65.9)
- moved TP9 2.54 mm to (108.1, 89.4)
- moved TP10 2.48 mm to (129.2, 81.1)
- moved TP22 2.48 mm to (126.6, 81.1)
- moved J11 2.42 mm to (97.9, 94.4), turned to 270 degrees
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Connections:
- F1 pad 1: Vin -> /measurement/VC16
- F17 pad 1: GND -> Vin
- F17 pad 2: Net-(F17-Pad2) -> Net-(F1-Pad2)
- J11 pad 1: GND -> /measurement/T1
- J11 pad 2: /measurement/T1 -> GND
- J12 pad 1: GND -> /measurement/T2
- J12 pad 2: /measurement/T2 -> GND
- J13 pad 1: GND -> /measurement/T3
- J13 pad 2: /measurement/T3 -> GND
- J3 pad 1: GND -> +5V
- J3 pad 2: /EN_OUT -> /SCL1
- J3 pad 3: /EN_IN -> /SDA1
- J3 pad 4: /SDA -> /EN_CHG
- J3 pad 5: /SCL -> /EN_DSGA
- J3 pad 6: +5V -> GND
- J6 pad 17: Vin -> /measurement/VC16
- J8 pad 9: Net-(F17-Pad2) -> GND
- R5 pad 2: /SCL -> /SCL2
- R6 pad 2: /SDA -> /SDA2
- R7 pad 2: Vin -> /measurement/VC16
- R8 pad 2: Vin -> /measurement/VC16
- U2 pad 2: /EN_IN -> /EN_DSGA
- U2 pad 21: /SDA -> /SDA2
- U2 pad 22: /SCL -> /SCL2
- U2 pad 3: /EN_OUT -> /EN_CHG
- U2 pad 31: Net-(TP23-Pad1) -> /PI_ON
- U2 pad 38: Net-(TP20-Pad1) -> /CS_B
- U2 pad 39: /PI_ON -> /CS_A
- U2 pad 4: Net-(TP6-Pad1) -> /EN_DSGB
- U2 pad 40: /CS_B -> /DSB
- U2 pad 41: /CS_A -> /DSA
- U2 pad 45: /DSB -> /SDA1
- U2 pad 46: /DSA -> /SCL1
- U3 pad 10: /SCL -> /SCL2
- U3 pad 9: /SDA -> /SDA2
Routing:
- net /SDA: track 94.7 -> 0.00 mm, vias 4 -> 0
- net /SCL: track 93.8 -> 0.00 mm, vias 4 -> 0
- net Vin: track 243.4 -> 156.1 mm
- net GND: track 360.1 -> 445.8 mm, vias 4 -> 30
- net /SCL2: track 0.00 -> 61.1 mm, vias 0 -> 2
- net /SDA2: track 0.00 -> 60.3 mm, vias 0 -> 2
- net /SDA1: track 0.00 -> 42.4 mm
- net /SCL1: track 0.00 -> 39.8 mm, vias 0 -> 1
- net +5V: track 252.5 -> 292.1 mm, vias 6 -> 16
- net /EN_CHG: track 0.00 -> 36.5 mm, vias 0 -> 3
- net /measurement/VC16: track 0.00 -> 32.3 mm
- net /EN_DSGA: track 0.00 -> 23.2 mm, vias 0 -> 2
- net /EN_DSGB: track 0.00 -> 19.8 mm, vias 0 -> 2
- net /EN_IN: track 16.3 -> 0.00 mm, vias 2 -> 0
- net /EN_OUT: track 16.1 -> 0.00 mm, vias 2 -> 0
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- added copper zone on B.Cu, net GND
Other:
- board text added: "3.3V Power Supply"
- board text added: "5V Power Supply"
- board text added: "5VA Filter"
- board text added: "AIN2"
- board text added: "AIN3"
- board text added: "Pi Zero Filter & Switch"
- board text added: "Temperature Sense"
- board text added: "V0"
- board text added: "V1"
- board text added: "V10"
- board text added: "V11"
- board text added: "V12"
- board text added: "V13"
- board text added: "V14"
- board text added: "V15"
- board text added: "V16"
- board text added: "V2"
- board text added: "V3"
- board text added: "V4"
- board text added: "V5"
- board text added: "V6"
- board text added: "V7"
- board text added: "V8"
- board text added: "V9"
- board text added: "Voltage Sensing"
- board text removed: "3V3"
- board text removed: "5V"
- board text removed: "5VA"

Commit message: v0.1
Parts:
- removed D3: BAT46, Diode_THT:D_DO-35_SOD27_P7.62mm_Horizontal
- added REF**: OSHW-Logo_5.7x6mm_SilkScreen, Symbol:OSHW-Logo_5.7x6mm_SilkScreen, F.Cu at (189.1, 99.9)
- D1: footprint Diode_THT:D_DO-35_SOD27_P7.62mm_Horizontal -> Diode_SMD:D_SMB-SMC_Universal_Handsoldering
- moved D1 4.86 mm to (187.0, 115.2)
- moved C27 0.38 mm to (133.1, 112.4), turned to 270 degrees
Routing:
- net GND: track 445.8 -> 480.8 mm, vias 30 -> 37
- net /USB_DM: track 17.1 -> 28.3 mm
- net Net-(R19-Pad2): track 26.7 -> 29.2 mm
- net Net-(C27-Pad1): track 7.43 -> 6.21 mm
- net Net-(R21-Pad2): track 28.4 -> 29.4 mm
- net /SCL2: track 61.1 -> 60.4 mm
- net Vin: track 156.1 -> 156.7 mm
Other:
- board text added: "Controller Module | Version 0.1 | 2019-11-11"
- board text removed: "Controller Module | Version 0.1"
