File: main-board/main-board.sch (KiCad schematic (older format))
At the start: 73 parts, among them J1 Conn_01x08_Male, J10 Raspberry_Pi_2_3, J11 T1, J12 T2, J13 T3, J2 USB_B, J3 Ext 5V, J4 Power Supply, J5 SWD, J6 Conn_01x17_Female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

Commit message: multiple changes
Parts:
- removed C5: 1u, Capacitor_SMD:C_0805_2012Metric, symbol Device:C
- removed D1: 68V, Diode_THT:D_DO-35_SOD27_P7.62mm_Horizontal, symbol Device:D_Schottky
- removed D4: 1N4733, Diode_THT:D_DO-41_SOD81_P7.62mm_Horizontal, symbol Device:D_Zener
- removed F18, F19: 2A, Resistor_SMD:R_2512_6332Metric, symbol Device:Fuse_Small
- removed J3: Ext 5V, TerminalBlock_RND:TerminalBlock_RND_205-00288_1x03_P5.08mm_Horizontal, symbol Connector:Screw_Terminal_01x03
- removed J4: Power Supply, TerminalBlock_RND:TerminalBlock_RND_205-00287_1x02_P5.08mm_Horizontal, symbol Connector:Screw_Terminal_01x02
- removed PS1: StepDownModule, footprints:LM2596HV_Module, symbol main-board:StepDownModule
- removed R1, R2: 20R, Resistor_SMD:R_0805_2012Metric, symbol Device:R_Small
- removed SW1: SW_DIP_x01, Button_Switch_THT:SW_Slide_1P2T_CK_OS102011MS2Q, symbol Switch:SW_DIP_x01
- added C31, C5: 22u, Capacitor_SMD:C_1206_3216Metric, symbol Device:C_Small
- added D1: 68V, Diode_THT:D_DO-35_SOD27_P7.62mm_Horizontal, symbol Device:D_Zener_Small
- added J3: ShuntBoard, TerminalBlock_4Ucon:TerminalBlock_4Ucon_1x06_P3.50mm_Horizontal, symbol Connector:Conn_01x06_Female
- added JP2: Bootloader, Jumper:SolderJumper-2_P1.3mm_Open_RoundedPad1.0x1.5mm, symbol Jumper:SolderJumper_2_Open
- added L2: BLM21PG600SN1, Inductor_SMD:L_1210_3225Metric_Pad1.42x2.65mm_HandSolder, symbol Device:L_Small
- added Q1: AO3400, Package_TO_SOT_SMD:SOT-23, symbol Device:Q_NMOS_GSD
- added R24, R25: 10k, Resistor_SMD:R_0805_2012Metric, symbol Device:R_Small
- added TP10, TP9: GND, TestPoint:TestPoint_THTPad_2.0x2.0mm_Drill1.0mm, symbol Connector:TestPoint
- J1: value Conn_01x08_Male -> ModuleConnector
- J11, J12, J13: footprint TerminalBlock_MetzConnect:TerminalBlock_MetzConnect_Type059_RT06303HBWC_1x03_P3.50mm_Horizontal -> TerminalBlock_MetzConnect:TerminalBlock_MetzConnect_Type059_RT06302HBWC_1x02_P3.50mm_Horizontal; symbol Connector:Screw_Terminal_01x03 -> Connector:Screw_Terminal_01x02
- J6: value Conn_01x17_Female -> Battery
- L1: value 10nH -> LQH3C 220u; footprint (none) -> Inductor_SMD:L_1210_3225Metric_Pad1.42x2.65mm_HandSolder
- PB0: renamed from TP9; value PB6 -> PB8; footprint TestPoint:TestPoint_THTPad_2.5x2.5mm_Drill1.2mm -> TestPoint:TestPoint_THTPad_2.0x2.0mm_Drill1.0mm
- PB1: renamed from TP10; value PB7 -> PB9; footprint TestPoint:TestPoint_THTPad_2.5x2.5mm_Drill1.2mm -> TestPoint:TestPoint_THTPad_2.0x2.0mm_Drill1.0mm
- R4: value 120R -> 62R
- TP13, TP14, TP15, TP16, TP17, TP18, TP19, TP2, TP21, TP22, TP23, TP3, TP6: footprint TestPoint:TestPoint_THTPad_2.5x2.5mm_Drill1.2mm -> TestPoint:TestPoint_THTPad_2.0x2.0mm_Drill1.0mm
- TP20: value PA3 -> PA15; footprint TestPoint:TestPoint_THTPad_2.5x2.5mm_Drill1.2mm -> TestPoint:TestPoint_THTPad_2.0x2.0mm_Drill1.0mm
- TP4: value PC13 -> 5V; footprint TestPoint:TestPoint_THTPad_2.5x2.5mm_Drill1.2mm -> TestPoint:TestPoint_THTPad_2.0x2.0mm_Drill1.0mm
- TP5: value PC14 -> 3V3; footprint TestPoint:TestPoint_THTPad_2.5x2.5mm_Drill1.2mm -> TestPoint:TestPoint_THTPad_2.0x2.0mm_Drill1.0mm
- TP7: value PB4 -> GND; footprint TestPoint:TestPoint_THTPad_2.5x2.5mm_Drill1.2mm -> TestPoint:TestPoint_THTPad_2.0x2.0mm_Drill1.0mm
- TP8: value PB5 -> PB2; footprint TestPoint:TestPoint_THTPad_2.5x2.5mm_Drill1.2mm -> TestPoint:TestPoint_THTPad_2.0x2.0mm_Drill1.0mm
Connections:
- net measurement/VC16 is gone; now on net Vin: F1.1, J6.17 (Pin_17)
- net +3V3: now also TP5.1, R25.1
- net +5V: now also TP4.1, J3.6 (Pin_6), L2.2; no longer J11.3 (Pin_3), J12.3 (Pin_3), J13.3 (Pin_3)
- net +5VA: now also C5.1
- net CS_A: now also U2.41 (PB5); no longer U2.18 (PB0)
- net CS_B: now also U2.40 (PB4); no longer U2.19 (PB1)
- net DSA: now also U2.46 (PB9); no longer U2.39 (PB3)
- net DSB: now also U2.45 (PB8); no longer U2.20 (PB2)
- net GND: now also TP7.1, C31.2, C5.2, D1.2 (A), J3.1 (Pin_1), JP2.1 (A), Q1.2 (S), R24.2, TP10.1, TP9.1; no longer J10.6 (GND)
- net SCL: now also J3.5 (Pin_5)
- net SDA: now also J3.4 (Pin_4)
- net USB_DM: now also J2.2 (D-)
- net USB_DP: now also J2.3 (D+)
- net Vin: now also D1.1 (K)
- net at TP20.1: now also U2.38 (PA15); no longer U2.13 (PA3)
- net EN_IN: now reaches U2.2 (PC13)
- net EN_IN: now also J3.3 (Pin_3); no longer TP4.1
- net EN_OUT: now reaches U2.3 (PC14)
- net EN_OUT: now also J3.2 (Pin_2); no longer TP5.1
- net LED: now reaches R4.1
- net LED: now also U2.13 (PA3); no longer U2.38 (PA15)
- net at TP8.1: now also U2.20 (PB2); no longer U2.41 (PB5)
- net at PB0.1: now also U2.18 (PB0); no longer U2.42 (PB6)
- net at PB1.1: now also U2.19 (PB1); no longer U2.43 (PB7)
- net at TP1.1, U2.44 (BOOT0): now also JP2.2 (B), R25.2
- net UART_TX: now reaches J10.10 (GPIO15/RXD)
- net UART_TX: now also U2.42 (PB6)
- net at J10.2 (5V), J10.4 (5V): now also C31.1, L2.1
- net UART_RX: now reaches J10.8 (GPIO14/TXD)
- net UART_RX: now also U2.43 (PB7)
- net at J10.9 (GND): now also Q1.3 (D)
- net PI_SCL: no longer names the net of J10.5 (SCL/GPIO3)
- net PI_SCL: no longer U2.45 (PB8)
- net PI_SDA: no longer names the net of J10.3 (SDA/GPIO2)
- net PI_SDA: no longer U2.46 (PB9)
- new net PI_ON: Q1.1 (G), R24.1, U2.39 (PB3)
Other:
- moved on the sheet: C28, D2, D3, J1, J10, J2, J5, L1, PB0, PB1, R4, TP1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

Commit message: multiple changes
Parts:
- removed D3: BAT46, Diode_THT:D_DO-35_SOD27_P7.62mm_Horizontal, symbol Device:D_Schottky_Small
- removed TP20: PA15, TestPoint:TestPoint_THTPad_2.0x2.0mm_Drill1.0mm, symbol Connector:TestPoint
- removed TP23: PA10, TestPoint:TestPoint_THTPad_2.0x2.0mm_Drill1.0mm, symbol Connector:TestPoint
- removed TP6: PC15, TestPoint:TestPoint_THTPad_2.0x2.0mm_Drill1.0mm, symbol Connector:TestPoint
- added H1, H2, H3, H4: MountingHole, MountingHole:MountingHole_3.2mm_M3_DIN965_Pad, symbol Mechanical:MountingHole_Pad
- added J4: ShuntBoard, Connector_JST:JST_XH_S6B-XH-A_1x06_P2.50mm_Horizontal, symbol Connector:Conn_01x06_Female
- added R32, R33: 2k2, Resistor_SMD:R_0805_2012Metric, symbol Device:R_Small
- F1, F10, F11, F12, F13, F14, F15, F16, F2, F3, F4, F5, F6, F7, F8, F9: footprint Resistor_SMD:R_2512_6332Metric -> Resistor_SMD:R_1812_4532Metric_Pad1.30x3.40mm_HandSolder
- F17: value 2A -> 1A; footprint Resistor_SMD:R_2512_6332Metric -> Resistor_SMD:R_1812_4532Metric_Pad1.30x3.40mm_HandSolder
- J11, J12, J13: footprint TerminalBlock_MetzConnect:TerminalBlock_MetzConnect_Type059_RT06302HBWC_1x02_P3.50mm_Horizontal -> Connector_JST:JST_XH_S2B-XH-A_1x02_P2.50mm_Horizontal; symbol Connector:Screw_Terminal_01x02 -> Connector:Conn_01x02_Male
- J2: value USB_B -> USB
- J3: footprint TerminalBlock_4Ucon:TerminalBlock_4Ucon_1x06_P3.50mm_Horizontal -> Connector_JST:JST_XH_S6B-XH-A_1x06_P2.50mm_Horizontal
- JP2: value Bootloader -> Boot
- L2: footprint Inductor_SMD:L_1210_3225Metric_Pad1.42x2.65mm_HandSolder -> Inductor_SMD:L_0805_2012Metric_Pad1.15x1.40mm_HandSolder
Connections:
- net +3V3: now also R32.1, R33.1
- net +5V: now also J3.1 (Pin_1), J4.1 (Pin_1); no longer J3.6 (Pin_6)
- net CS_A: now also U2.39 (PB3); no longer U2.41 (PB5)
- net CS_B: now also U2.38 (PA15); no longer U2.40 (PB4)
- net DSA: now also U2.41 (PB5); no longer U2.46 (PB9)
- net DSB: now also U2.40 (PB4); no longer U2.45 (PB8)
- net GND: now also J11.2 (Pin_2), J12.2 (Pin_2), J13.2 (Pin_2), J3.6 (Pin_6), J8.9 (Pin_9), J4.6 (Pin_6); no longer F17.1, J11.1 (Pin_1), J12.1 (Pin_1), J13.1 (Pin_1), J3.1 (Pin_1)
- net PI_ON: now also U2.31 (PA10); no longer U2.39 (PB3)
- net Vin: now also F17.1; no longer F1.1, J6.17 (Pin_17)
- net measurement/T1: now also J11.1 (Pin_1); no longer J11.2 (Pin_2)
- net measurement/T2: now also J12.1 (Pin_1); no longer J12.2 (Pin_2)
- net measurement/T3: now also J13.1 (Pin_1); no longer J13.2 (Pin_2)
- net at F17.2: now also F1.2, J7.1 (Pin_1); no longer J8.9 (Pin_9)
- net EN_DSGB: now reaches U2.4 (PC15)
- net EN_DSGB: now also J4.5 (Pin_5)
- net EN_IN renamed EN_DSGA
- net EN_DSGA: now also J3.5 (Pin_5); no longer J3.3 (Pin_3)
- net EN_OUT renamed EN_CHG
- net EN_CHG: now also J3.4 (Pin_4), J4.4 (Pin_4); no longer J3.2 (Pin_2)
- net SCL renamed SCL2
- net SCL2: no longer J3.5 (Pin_5)
- net SDA renamed SDA2
- net SDA2: no longer J3.4 (Pin_4)
- new net SCL1: J3.2 (Pin_2), J4.2 (Pin_2), R32.2, U2.46 (PB9)
- new net SDA1: J3.3 (Pin_3), J4.3 (Pin_3), R33.2, U2.45 (PB8)
- new net measurement/VC16: F1.1, J6.17 (Pin_17)
- no-connect marks 1 -> 5
Other:
- moved on the sheet: D1, J3

Commit message: v0.1
Parts:
- D1: footprint Diode_THT:D_DO-35_SOD27_P7.62mm_Horizontal -> Diode_SMD:D_SMB-SMC_Universal_Handsoldering
Changed lines of the file:
@@
 F 0 "D1" V 1254 1368 50  0000 L CNN
 F 1 "68V" V 1345 1368 50  0000 L CNN
-F 2 "Diode_THT:D_DO-35_SOD27_P7.62mm_Horizontal" V 1300 1300 50  0001 C CNN
+F 2 "Diode_SMD:D_SMB-SMC_Universal_Handsoldering" V 1300 1300 50  0001 C CNN
 F 3 "~" V 1300 1300 50  0001 C CNN
 	1    1300 1300
