File: switch-board/shunt-board.kicad_pcb (KiCad board)
At the start: 2 copper layers, 92 x 95 mm, 52 parts, among them J1 Connector, J2 BAT-, J3 BAT+, J4 C-, J5 L-, J6 OUT+, Q1 TPH1R306PL, Q2 TPH1R306PL, Q3 TPH1R306PL, Q4 TPH1R306PL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

Commit message: v0.1
Parts:
- C1: footprint Capacitor_THT:CP_Radial_D6.3mm_P2.50mm -> Capacitor_SMD:C_0805_2012Metric_Pad1.15x1.40mm_HandSolder
- moved C1 2.73 mm to (176.5, 100.3)
Routing:
- net GND: track 11.8 -> 8.45 mm, vias 5 -> 6
Other:
- board text added: "Switch Module | Version 0.1 | 2019-11-11"
- board text removed: "Switch Module | Version 0.1"
