File: switch-board/shunt-board.sch (KiCad schematic (older format))
At the start: 45 parts, among them J1 Connector, J2 BAT-, J3 BAT+, J4 C-, J5 L-, J6 OUT+, U1 BQ76200, U2 ADS1115IDGS

Commit message: v0.1
Parts:
- C1: footprint Capacitor_THT:CP_Radial_D6.3mm_P2.50mm -> Capacitor_SMD:C_0805_2012Metric_Pad1.15x1.40mm_HandSolder
Changed lines of the file:
@@
 F 0 "C1" H 4392 2396 50  0000 L CNN
 F 1 "10n 63V" H 4392 2305 50  0000 L CNN
-F 2 "Capacitor_THT:CP_Radial_D6.3mm_P2.50mm" H 4300 2350 50  0001 C CNN
+F 2 "Capacitor_SMD:C_0805_2012Metric_Pad1.15x1.40mm_HandSolder" H 4300 2350 50  0001 C CNN
 F 3 "~" H 4300 2350 50  0001 C CNN
 	1    4300 2350
